File: kicad/modules/hellen1-wbo/hellen1-wbo.kicad_sch (KiCad schematic)
At the start: 65 parts, among them J600 Conn_02x03_Odd_Even, M600 Module-wbo-0.5, Q600 BTS3028, Q601 VNP28N04-E, U600 MCP6004, U601 AD8628, U602 STM32F042K6Tx, U603 REF3033, U604 XC6206P332MR, U605 TJA1051T/3/1J

Commit message: new
Other:
- company: rusefi.com -> gerefi.com
Changed lines of the file:
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@@
     (date "2021-09-28")
     (rev "0.5")
-    (company "rusefi.com")
+    (company "gerefi.com")
   )
   (junction (at 135.89 30.48) (diameter 1.016) (color 0 0 0 0)
