File: tests/hellen1test.kicad_sch (KiCad schematic)
At the start: 8 parts, among them M1 Module-can-0.1, P1 Pad, P2 Pad, P3 Pad, P4 Pad, P5 Pad, P6 Pad, P7 Pad

Commit message: new
Other:
- note added: "https://gerefi.com/"
- note added: "https://github.com/gerefi2-git/hellen-one/wiki"
- note removed: "https://github.com/andreika-git/hellen-one/wiki"
- note removed: "https://rusefi.com/"
Changed lines of the file:
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@@
     )
   )
-  (text "https://rusefi.com/" (at 213.36 180.34 180)
+  (text "https://gerefi.com/" (at 213.36 180.34 180)
     (effects (font (size 1.27 1.27)) (justify right bottom))
   )
-  (text "https://github.com/andreika-git/hellen-one/wiki" (at 275.59 180.34 180)
+  (text "https://github.com/gerefi2-git/hellen-one/wiki" (at 275.59 180.34 180)
     (effects (font (size 1.27 1.27)) (justify right bottom))
   )
